File: Servo_Board/Servo_Board.kicad_sch (KiCad schematic)
At the start: 44 parts

Commit message: Updated Schematic
Parts:
- removed R?: 8 Ohm, symbol Device:R_Small
- removed R?: 4 Ohm, symbol Device:R_Small
- added C? (x2): 100u, symbol pspice:CAP
- added C? (x3): 2.2u, symbol pspice:CAP
- added C?: .2 uF, symbol Device:C_Small
- added C?: 70p, symbol pspice:CAP
- added D?: DIODE, symbol pspice:DIODE
- added D?: 300V Schottky, symbol Device:D_Schottky
- added DPOT?: 10k, symbol Drone-Circuit-rescue:Digital_Pot-Project_Library
- added L?: 5 uH, symbol pspice:INDUCTOR
- added M?: NMOS, symbol pspice:MNMOS
- added R?: 400, symbol pspice:R
- added R?: 60k, symbol Device:R
- added U? (x2): 5V linear regulator, Package_TO_SOT_SMD:SOT-223-3_TabPin2, symbol Regulator_Linear:AMS1117-5.0
- added U?: 555, symbol Timer:LM555xM
Connections:
- net GND: now also C?.1, C?.1, C?.2, C?.2, C?.2, C?.2, D?.2 (A), DPOT?.4 (VSS), M?.4 (B), R?.2, U?.1 (GND), U?.1 (GND)
- net ~14V: now also M?.1 (D), U?.3 (VI)
- net 12V Output renamed 12V
- net 5V Output renamed 5V2
- net 5V2: now also C?.1, R?.1, U?.2 (VO)
- net 6V Output renamed 6V
- new net: D?.1 (K), M?.2 (G), U?.3 (Q)
- new net: D?.2 (A), DPOT?.7 (P0B)
- new net: D?.1 (K), L?.1, M?.3 (S)
- new net: DPOT?.5 (P0A), R?.2
- new net: C?.1, DPOT?.6 (P0W), U?.2 (TR), U?.6 (THR)
- new net: C?.2, C?.2, L?.2, U?.3 (VI)
- new net: R?.1, U?.7 (DIS)
- new net 0: C?.2, U?.1 (GND)
- new net 5V1: C?.1, C?.1, C?.1, DPOT?.8 (VDD), U?.2 (VO), U?.4 (R), U?.8 (VCC)
- new net DP_CE0: DPOT?.1 (~{CS})
- new net DP_MOSI: DPOT?.3 (SDI/SDO)
- new net DP_SCLK: DPOT?.2 (SCK)
Other:
- note added: "We need to check if this linear regulator can handle 14V"
