File: Servo_Board/Power_Board.kicad_sch (KiCad schematic)
At the start: 59 parts

Commit message: Created footprint for ADC, tossed it in unconnected
Parts:
- added ADC?: ADS1115, Custom_Footprints:ADS1115-16Bit, symbol Custom_Symbols:ADS1115
