File: Servo_Board/Power_Board.kicad_sch (KiCad schematic)
At the start: 47 parts

Commit message: footprint
Parts:
- added U?: raspberry_pi, SARP:Raspberry Pi, symbol custom:raspberry_pi
Changed lines of the file:
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@@
     (pin "1")
+  )
+  (symbol (lib_id "custom:raspberry_pi") (at 25.4 157.48 0) (unit 1)
+    (in_bom yes) (on_board yes) (fields_autoplaced)
+    (property "Reference" "U?" (id 0) (at 34.29 156.2099 0)
+      (effects (font (size 1.27 1.27)) (justify left))
+    )
+    (property "Value" "raspberry_pi" (id 1) (at 34.29 158.7499 0)
+      (effects (font (size 1.27 1.27)) (justify left))
+    )
+    (property "Footprint" "SARP:Raspberry Pi" (id 2) (at 25.4 157.48 0)
+      (effects (font (size 1.27 1.27)) hide)
+    )
+    (property "Datasheet" "" (id 3) (at 25.4 157.48 0)
+      (effects (font (size 1.27 1.27)) hide)
+    )
   )
   (symbol (lib_id "Device:R_Small") (at 29.21 92.71 90) (unit 1)
@@
       (reference "R?") (unit 1) (value "60k") (footprint "")
     )
+    (path "/2d809e94-e752-4170-b68a-f6d9b51272b9"
+      (reference "U?") (unit 1) (value "raspberry_pi") (footprint "SARP:Raspberry Pi")
+    )
     (path "/63ce923e-7fea-4015-b4ae-cf8da31bbf6f"

Commit message: added components
Parts:
- added U?: Small_thing, SARP:small thing, symbol SARP:Small_thing
- added U?: Radio_Thing, SARP:radio thing, symbol SARP:Radio_Thing
Changed lines of the file:
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@@
     )
+  )
+  (symbol (lib_id "SARP:Small_thing") (at 36.83 184.15 0) (unit 1)
+    (in_bom yes) (on_board yes) (fields_autoplaced)
+    (property "Reference" "U?" (id 0) (at 60.96 182.8799 0)
+      (effects (font (size 1.27 1.27)) (justify left))
+    )
+    (property "Value" "Small_thing" (id 1) (at 60.96 185.4199 0)
+      (effects (font (size 1.27 1.27)) (justify left))
+    )
+    (property "Footprint" "SARP:small thing" (id 2) (at 36.83 184.15 0)
+      (effects (font (size 1.27 1.27)) hide)
+    )
+    (property "Datasheet" "" (id 3) (at 36.83 184.15 0)
+      (effects (font (size 1.27 1.27)) hide)
+    )
+    (pin "1")
+    (pin "2")
+    (pin "3")
+    (pin "4")
   )
   (symbol (lib_id "Device:R_Small") (at 29.21 92.71 90) (unit 1)
@@
     (pin "1")
     (pin "2")
+  )
+  (symbol (lib_id "SARP:Radio_Thing") (at 82.55 162.56 0) (unit 1)
+    (in_bom yes) (on_board yes) (fields_autoplaced)
+    (property "Reference" "U?" (id 0) (at 101.6 160.6549 0)
+      (effects (font (size 1.27 1.27)) (justify left))
+    )
+    (property "Value" "Radio_Thing" (id 1) (at 101.6 163.1949 0)
+      (effects (font (size 1.27 1.27)) (justify left))
+    )
+    (property "Footprint" "SARP:radio thing" (id 2) (at 101.6 165.7349 0)
+      (effects (font (size 1.27 1.27)) (justify left))
+    )
+    (property "Datasheet" "" (id 3) (at 82.55 162.56 0)
+      (effects (font (size 1.27 1.27)) hide)
+    )
   )
   (symbol (lib_id "power:GND") (at 252.73 62.23 270) (unit 1)
@@
       (reference "U?") (unit 1) (value "raspberry_pi") (footprint "SARP:Raspberry Pi")
     )
+    (path "/2fad1abc-4c32-4010-9ef6-3e0f8b7321e3"
+      (reference "U?") (unit 1) (value "Small_thing") (footprint "SARP:small thing")
+    )
     (path "/63ce923e-7fea-4015-b4ae-cf8da31bbf6f"
       (reference "U?") (unit 1) (value "Adafruit_IMU_BNO055") (footprint "")
     )
+    (path "/6715ed73-4a44-4072-9696-f066d9697e23"
+      (reference "U?") (unit 1) (value "Radio_Thing") (footprint "SARP:radio thing")
+    )
     (path "/7b539afc-805f-494c-b8a6-cdda86fbd90a"
