File: Servo_Board/Power_Board.kicad_sch (KiCad schematic)
At the start: 48 parts

Commit message: PDR update
Parts:
- removed U?: 5V linear regulator, Package_TO_SOT_SMD:SOT-223-3_TabPin2, symbol Regulator_Linear:AMS1117-5.0
- added U?: AMS1117-3.3, Package_TO_SOT_SMD:SOT-223-3_TabPin2, symbol Regulator_Linear:AMS1117-3.3
Connections:
- net 0: now also U?.1 (GND)
- net ~14V: now also U?.3 (VI)
- net 5V1 renamed 3V3_1
- net 3V3_1: now also U?.2 (VO)
Other:
- note removed: "We need to check if this linear regulator can handle 14V"
Changed lines of the file:
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@@
-    (stroke (width 0) (type default) (color 0 0 0 0))
-  )
-  (polyline (pts (xy 107.95 19.05) (xy 107.95 21.59))
     (stroke (width 0) (type default) (color 0 0 0 0))
   )
@@
     (stroke (width 0) (type default) (color 0 0 0 0))
   )
-  (polyline (pts (xy 86.36 19.05) (xy 107.95 19.05))
-    (stroke (width 0) (type default) (color 0 0 0 0))
-  )
   (wire (pts (xy 233.68 52.07) (xy 223.52 52.07))
     (stroke (width 0) (type default) (color 0 0 0 0))
@@
   )
   (wire (pts (xy 129.54 44.45) (xy 123.19 44.45))
-    (stroke (width 0) (type default) (color 0 0 0 0))
-  )
-  (polyline (pts (xy 86.36 16.51) (xy 86.36 19.05))
     (stroke (width 0) (type default) (color 0 0 0 0))
   )
@@
     (effects (font (size 1.27 1.27)) (justify left bottom))
   )
-  (text "We need to check if this linear regulator can handle 14V"
-    (at 52.07 16.51 0)
+  (text "Sensor board" (at 210.82 15.24 0)
     (effects (font (size 1.27 1.27)) (justify left bottom))
   )
-  (text "Sensor board" (at 210.82 15.24 0)
+  (label "3V3_1" (at 157.48 49.53 0)
+    (effects (font (size 1.27 1.27)) (justify left bottom))
+  )
+  (label "3V3_1" (at 120.65 21.59 90)
+    (effects (font (size 1.27 1.27)) (justify left bottom))
+  )
+  (label "3V3_1" (at 115.57 67.31 90)
+    (effects (font (size 1.27 1.27)) (justify left bottom))
+  )
+  (label "3V3_1" (at 144.78 29.21 90)
     (effects (font (size 1.27 1.27)) (justify left bottom))
   )
@@
     (property "Intersheet References" "${INTERSHEET_REFS}" (id 0) (at -50.165 417.83 0)
       (effects (font (size 1.27 1.27)) hide)
-    )
-  )
-  (global_label "5V1" (shape output) (at 120.65 20.32 90) (fields_autoplaced)
-    (effects (font (size 1.27 1.27)) (justify left))
-    (property "Intersheet References" "${INTERSHEET_REFS}" (id 0) (at 120.5706 14.3993 90)
-      (effects (font (size 1.27 1.27)) (justify left) hide)
     )
   )
@@
     )
   )
-  (global_label "5V1" (shape input) (at 115.57 66.04 90) (fields_autoplaced)
-    (effects (font (size 1.27 1.27)) (justify left))
-    (property "Intersheet References" "${INTERSHEET_REFS}" (id 0) (at -40.64 415.29 0)
-      (effects (font (size 1.27 1.27)) hide)
-    )
-  )
   (global_label "6V" (shape output) (at 69.85 80.01 90) (fields_autoplaced)
     (effects (font (size 1.27 1.27)) (justify left))
@@
     )
   )
-  (global_label "5V1" (shape input) (at 144.78 27.94 90) (fields_autoplaced)
-    (effects (font (size 1.27 1.27)) (justify left))
-    (property "Intersheet References" "${INTERSHEET_REFS}" (id 0) (at 265.43 -353.06 0)
-      (effects (font (size 1.27 1.27)) hide)
-    )
-  )
   (global_label "~14V" (shape input) (at 13.97 22.86 90) (fields_autoplaced)
     (effects (font (size 1.27 1.27)) (justify left))
@@
     )
   )
-  (global_label "5V1" (shape input) (at 158.75 49.53 0) (fields_autoplaced)
-    (effects (font (size 1.27 1.27)) (justify left))
-    (property "Intersheet References" "${INTERSHEET_REFS}" (id 0) (at -190.5 -106.68 0)
-      (effects (font (size 1.27 1.27)) hide)
-    )
-  )
   (global_label "12V" (shape output) (at 69.85 113.03 90) (fields_autoplaced)
     (effects (font (size 1.27 1.27)) (justify left))
@@
     (pin "1")
     (pin "2")
+  )
+  (symbol (lib_id "Regulator_Linear:AMS1117-3.3") (at 111.76 24.13 0) (unit 1)
+    (in_bom yes) (on_board yes) (fields_autoplaced)
+    (property "Reference" "U?" (id 0) (at 111.76 16.51 0))
+    (property "Value" "AMS1117-3.3" (id 1) (at 111.76 19.05 0))
+    (property "Footprint" "Package_TO_SOT_SMD:SOT-223-3_TabPin2" (id 2) (at 111.76 19.05 0)
+      (effects (font (size 1.27 1.27)) hide)
+    )
+    (property "Datasheet" "http://www.advanced-monolithic.com/pdf/ds1117.pdf" (id 3) (at 114.3 30.48 0)
+      (effects (font (size 1.27 1.27)) hide)
+    )
+    (pin "1")
+    (pin "2")
+    (pin "3")
   )
   (symbol (lib_id "power:GND") (at 26.67 59.69 270) (unit 1)
@@
     (pin "2")
   )
-  (symbol (lib_id "Regulator_Linear:AMS1117-5.0") (at 111.76 24.13 0) (unit 1)
-    (in_bom yes) (on_board yes) (fields_autoplaced)
-    (property "Reference" "U?" (id 0) (at 110.4899 20.32 90)
-      (effects (font (size 1.27 1.27)) (justify left))
-    )
-    (property "Value" "5V linear regulator" (id 1) (at 113.0299 20.32 90)
-      (effects (font (size 1.27 1.27)) (justify left))
-    )
-    (property "Footprint" "Package_TO_SOT_SMD:SOT-223-3_TabPin2" (id 2) (at 111.76 19.05 0)
-      (effects (font (size 1.27 1.27)) hide)
-    )
-    (property "Datasheet" "http://www.advanced-monolithic.com/pdf/ds1117.pdf" (id 3) (at 114.3 30.48 0)
-      (effects (font (size 1.27 1.27)) hide)
-    )
-    (pin "1")
-    (pin "2")
-    (pin "3")
-  )
   (symbol (lib_id "Device:C_Small") (at 41.91 110.49 0) (unit 1)
     (in_bom yes) (on_board yes) (fields_autoplaced)
@@
       (reference "U?") (unit 1) (value "raspberry_pi") (footprint "SARP:Raspberry Pi")
     )
+    (path "/47776730-c5b5-411b-84ad-524c46256894"
+      (reference "U?") (unit 1) (value "AMS1117-3.3") (footprint "Package_TO_SOT_SMD:SOT-223-3_TabPin2")
+    )
     (path "/63ce923e-7fea-4015-b4ae-cf8da31bbf6f"
       (reference "U?") (unit 1) (value "Adafruit_IMU_BNO055") (footprint "")
@@
       (reference "U?") (unit 1) (value "6V linear regulator") (footprint "Package_SO:HTSOP-8-1EP_3.9x4.9mm_P1.27mm_EP2.4x3.2mm")
     )
-    (path "/95ecd73d-7219-4e2b-8504-3174bfd30355"
-      (reference "U?") (unit 1) (value "5V linear regulator") (footprint "Package_TO_SOT_SMD:SOT-223-3_TabPin2")
-    )
     (path "/daac08ec-05c7-4ce4-a956-343d6bb3eecd"
