File: Servo_Board/Flight_Computer/Flight_Computer.kicad_sch (KiCad schematic)
At the start: 17 parts

Commit message: g
Other:
- note added: "PC to laptop git test"
Changed lines of the file:
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@@
+    (effects (font (size 1.27 1.27)) (justify left bottom))
+  )
+  (text "PC to laptop git test" (at 19.05 165.1 0)
     (effects (font (size 1.27 1.27)) (justify left bottom))
   )

Commit message: Update Flight_Computer.kicad_sch
Parts:
- added U?: AMS1117-3.3, Package_TO_SOT_SMD:SOT-223-3_TabPin2, symbol Regulator_Linear:AMS1117-3.3
Changed lines of the file:
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@@
     (pin "4")
+  )
+  (symbol (lib_id "Regulator_Linear:AMS1117-3.3") (at 218.44 33.02 0) (unit 1)
+    (in_bom yes) (on_board yes) (fields_autoplaced)
+    (property "Reference" "U?" (id 0) (at 218.44 25.4 0))
+    (property "Value" "AMS1117-3.3" (id 1) (at 218.44 27.94 0))
+    (property "Footprint" "Package_TO_SOT_SMD:SOT-223-3_TabPin2" (id 2) (at 218.44 27.94 0)
+      (effects (font (size 1.27 1.27)) hide)
+    )
+    (property "Datasheet" "http://www.advanced-monolithic.com/pdf/ds1117.pdf" (id 3) (at 220.98 39.37 0)
+      (effects (font (size 1.27 1.27)) hide)
+    )
+    (pin "1")
+    (pin "2")
+    (pin "3")
   )
   (symbol (lib_id "Device:C") (at 104.14 31.75 0) (unit 1)
@@
       (reference "U?") (unit 1) (value "STM32F401CCU6") (footprint "Package_DFN_QFN:QFN-48-1EP_7x7mm_P0.5mm_EP5.6x5.6mm")
     )
+    (path "/7807eff4-fbe2-4048-bf33-9a3236b3d15c"
+      (reference "U?") (unit 1) (value "AMS1117-3.3") (footprint "Package_TO_SOT_SMD:SOT-223-3_TabPin2")
+    )
     (path "/6328ec20-8909-4d2e-9149-7750cecf5551"
