File: flight_computer/_autosave-Flight_Computer.kicad_sch (KiCad schematic)
At the start: 112 parts

Commit message: er
Parts:
- added R?: R, symbol Device:R
Changed lines of the file:
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@@
     (pin "1")
+  )
+  (symbol (lib_id "Device:R") (at 497.84 302.26 0) (unit 1)
+    (in_bom yes) (on_board yes) (fields_autoplaced)
+    (property "Reference" "R?" (id 0) (at 500.38 300.9899 0)
+      (effects (font (size 1.27 1.27)) (justify left))
+    )
+    (property "Value" "R" (id 1) (at 500.38 303.5299 0)
+      (effects (font (size 1.27 1.27)) (justify left))
+    )
+    (property "Footprint" "" (id 2) (at 496.062 302.26 90)
+      (effects (font (size 1.27 1.27)) hide)
+    )
+    (property "Datasheet" "~" (id 3) (at 497.84 302.26 0)
+      (effects (font (size 1.27 1.27)) hide)
+    )
+    (pin "1")
+    (pin "2")
   )
   (symbol (lib_id "power:GND") (at 419.1 68.58 0) (unit 1)
@@
       (reference "R?") (unit 1) (value "1ohm") (footprint "")
     )
+    (path "/bcc42a10-254e-4b59-974b-9e53229b341c"
+      (reference "R?") (unit 1) (value "R") (footprint "")
+    )
     (path "/c15cac80-936f-40cf-ab97-38fd3a7d70b9"
