File: flight_computer/Flight_Computer.kicad_sch (KiCad schematic)
At the start: 112 parts

Commit message: Update Flight_Computer.kicad_sch
Other:
- note added: "Hopefully this works"
Changed lines of the file:
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@@
     (effects (font (size 0.8 0.8)) (justify left bottom))
+  )
+  (text "Hopefully this works" (at 6.35 309.88 0)
+    (effects (font (size 1.27 1.27)) (justify left bottom))
   )
   (text "Micro SD Card connector" (at 116.84 55.88 0)

Commit message: bakerw
ignitor
Parts:
- added Male?: LEAD_MAIN1, symbol Connector:Conn_01x01_Male
- added Male?: LEAD_DROUG1, symbol Connector:Conn_01x01_Male
- added Male? (x2): Fire_Droug, symbol Connector:Conn_01x01_Male
- added Male? (x2): Male, symbol Connector:Conn_01x01_Male
- added Power_IN?, RPI_IN?: Cont_Droug, symbol Connector:Conn_01x01_Male
- added Q? (x2): FQP30N06L, Package_TO_SOT_THT:TO-220-3_Vertical, symbol Transistor_FET:FQP27P06
- added R? (x2): 10k, symbol Device:R
- added RPI_IN?: Fire_Main, symbol Connector:Conn_01x01_Male
- added RPI_IN?: Cont_Main, symbol Connector:Conn_01x01_Male
- added RPI_IN?: GND, symbol Connector:Conn_01x01_Male
- added VDiv1_? (x2), VDiv2_? (x2): ?Ohms, symbol Device:R
Connections:
- net GND: now also Male?.1 (Pin_1), Male?.1 (Pin_1), Q?.3 (S), Q?.3 (S), R?.2, R?.2, VDiv1_?.1, VDiv2_?.1
- new net: Male?.1 (Pin_1), Q?.2 (D), VDiv2_?.2
- new net: Male?.1 (Pin_1), Q?.2 (D), VDiv1_?.2
- new net Cont_Droug: RPI_IN?.2 (Pin_1), VDiv1_?.1, VDiv1_?.2
- new net Cont_Main: RPI_IN?.5 (Pin_1), VDiv2_?.1, VDiv2_?.2
- new net Fire_Droug: Q?.1 (G), R?.1, RPI_IN?.3 (Pin_1)
- new net Fire_Main: Q?.1 (G), R?.1, RPI_IN?.4 (Pin_1)
- new net VCC: Male?.1 (Pin_1), Power_IN?.2 (Pin_1)
Other:
- note added: "Igniter Droug"
- note added: "Igniter Main"

Commit message: resistors
Other:
- note added: "3.3V R1 = 1k R2 = 1.75k"
- note added: "6V R1 = 1k R2 = 4k"
Changed lines of the file:
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@@
+    (stroke (width 0) (type default) (color 0 0 0 0))
+  )
+  (polyline (pts (xy 106.68 -2.54) (xy 123.19 -2.54))
     (stroke (width 0) (type default) (color 0 0 0 0))
   )
@@
     (stroke (width 0) (type default) (color 0 0 0 0))
   )
+  (polyline (pts (xy 123.19 -2.54) (xy 123.19 -21.59))
+    (stroke (width 0) (type default) (color 0 0 0 0))
+  )
   (wire (pts (xy 64.77 54.61) (xy 52.07 54.61))
     (stroke (width 0) (type default) (color 0 0 0 0))
@@
     (stroke (width 0) (type default) (color 0 0 0 0))
   )
+  (polyline (pts (xy 106.68 -21.59) (xy 123.19 -21.59))
+    (stroke (width 0) (type default) (color 0 0 0 0))
+  )
   (wire (pts (xy 405.13 83.82) (xy 405.13 85.09))
     (stroke (width 0) (type default) (color 0 0 0 0))
@@
     (stroke (width 0) (type default) (color 0 0 0 0))
   )
+  (polyline (pts (xy 106.68 -21.59) (xy 106.68 -2.54))
+    (stroke (width 0) (type default) (color 0 0 0 0))
+  )
   (wire (pts (xy 128.27 256.54) (xy 128.27 260.35))
     (stroke (width 0) (type default) (color 0 0 0 0))
@@
   )
   (wire (pts (xy 215.9 97.79) (xy 123.19 97.79))
-    (stroke (width 0) (type default) (color 0 0 0 0))
-  )
-  (polyline (pts (xy 123.19 -10.16) (xy 124.46 -10.16))
     (stroke (width 0) (type default) (color 0 0 0 0))
   )
@@
     (effects (font (size 1.27 1.27)) (justify left bottom))
   )
+  (text "6V\nR1 = 1k\nR2 = 4k" (at 109.22 -3.81 0)
+    (effects (font (size 1.27 1.27)) (justify left bottom))
+  )
   (text "Find proper L and C values" (at 69.85 -26.67 0)
     (effects (font (size 1.27 1.27) (thickness 0.254) bold italic) (justify left bottom))
@@
     (effects (font (size 5 5)) (justify left bottom))
   )
+  (text "3.3V\nR1 = 1k\nR2 = 1.75k" (at 109.22 -12.7 0)
+    (effects (font (size 1.27 1.27)) (justify left bottom))
+  )
   (text "Redo exteranl pins and route radio pins and GPS pins"

Commit message: resistor
Parts:
- added R1 (x2): 1k, symbol Device:R
- added R2: 4k, symbol Device:R
- added R2: 1.75k, symbol Device:R
Connections:
- net +6V is gone; now on net +3V3: C?.1, J?.1 (Pin_1), J?.1 (Pin_1), J?.1 (Pin_1), L?.2, U?.4 (FB)
- net GND is gone; now on net +3V3: C?.1, C?.1, C?.1, C?.1, C?.1, C?.1, C?.1, C?.1, C?.1, C?.1, C?.1, C?.1, C?.1, C?.1, C?.1, C?.1, C?.2, C?.2, C?.2, C?.2, C?.2, C?.2, C?.2, C?.2, C?.2, C?.2, C?.2, C?.2, C?.2, C?.2, C?.2, C?.2, C?.2, C?.2, C?.2, C?.2, C?.2, C?.2, C?.2, C?.2, C?.2, C?.2, C?.2, C?.2, D?.2 (A), D?.2 (A), D?.2 (A), J?.2 (Pin_2), J?.4 (Pin_4), J?.6 (VSS), J?.A1 (GND), J?.A12 (GND), J?.A4 (VBUS), J?.A9 (VBUS), J?.B1 (GND), J?.B12 (GND), J?.B4 (VBUS), J?.B9 (VBUS), L?.2, Male?.1 (Pin_1), Male?.1 (Pin_1), Q?.3 (S), Q?.3 (S), R?.1, R?.1, R?.1, R?.1, R?.1, R?.2, R?.2, R?.2, R?.2, R?.2, R?.2, R?.2, SW?.1 (A), U?.1 (GND), U?.15 (GNDIO), U?.16 (GNDIO), U?.18 (COM2), U?.2 (GND), U?.23 (VSS), U?.25 (GNDIO), U?.3 (GND), U?.3 (GND), U?.3 (GND), U?.3 (VI), U?.32 (EXT_XOSC), U?.33 (GND_EP), U?.35 (VSS), U?.47 (VSS), U?.49 (VSS), U?.5 (~{ON}/OFF), U?.5 (~{ON}/OFF), U?.5 (~{ON}/OFF), U?.7 (GND), U?.8 (VSSA), U?.P$12 (GND@3), U?.P$19 (GND@4), U?.P$3 (GND@1), U?.P$8 (GND@2), VDiv1_?.1, VDiv2_?.1, X?.2, X?.4, Y?.2, Y?.4
- net +3V3: now also R1.2, R2.1, R2.1
- new net: R1.1, R2.2 (x2)
Changed lines of the file:
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@@
   (junction (at 405.13 83.82) (diameter 0) (color 0 0 0 0)
   )
+  (junction (at 85.09 -10.16) (diameter 0) (color 0 0 0 0)
+  )
   (junction (at 238.76 82.55) (diameter 0) (color 0 0 0 0)
   )
@@
   (junction (at 137.16 107.95) (diameter 0) (color 0 0 0 0)
   )
+  (junction (at 92.71 -76.2) (diameter 0) (color 0 0 0 0)
+  )
   (junction (at 82.55 121.92) (diameter 0) (color 0 0 0 0)
   )
@@
   (junction (at 133.35 74.93) (diameter 0) (color 0 0 0 0)
   )
+  (junction (at 85.09 -22.86) (diameter 0) (color 0 0 0 0)
+  )
   (junction (at 133.35 236.22) (diameter 0) (color 0 0 0 0)
   )
+  (junction (at 92.71 -17.78) (diameter 0) (color 0 0 0 0)
+  )
   (junction (at 71.12 243.84) (diameter 0) (color 0 0 0 0)
   )
@@
   (junction (at 80.01 121.92) (diameter 0) (color 0 0 0 0)
   )
+  (junction (at 90.17 -7.62) (diameter 0) (color 0 0 0 0)
+  )
   (junction (at 353.06 72.39) (diameter 0) (color 0 0 0 0)
   )
@@
   (junction (at 447.04 63.5) (diameter 0) (color 0 0 0 0)
   )
+  (junction (at 85.09 -81.28) (diameter 0) (color 0 0 0 0)
+  )
   (junction (at 234.95 59.69) (diameter 0) (color 0 0 0 0)
   )
@@
   (junction (at 210.82 127) (diameter 0) (color 0 0 0 0)
   )
+  (junction (at 85.09 -68.58) (diameter 0) (color 0 0 0 0)
+  )
   (junction (at 440.69 45.72) (diameter 0) (color 0 0 0 0)
   )
@@
     (stroke (width 0) (type default) (color 0 0 0 0))
   )
+  (wire (pts (xy 85.09 -68.58) (xy 85.09 -66.04))
+    (stroke (width 0) (type default) (color 0 0 0 0))
+  )
   (wire (pts (xy 41.91 -81.28) (xy 45.72 -81.28))
     (stroke (width 0) (type default) (color 0 0 0 0))
@@
     (stroke (width 0) (type default) (color 0 0 0 0))
   )
+  (wire (pts (xy 92.71 -76.2) (xy 92.71 -66.04))
+    (stroke (width 0) (type default) (color 0 0 0 0))
+  )
   (wire (pts (xy 447.04 76.2) (xy 443.23 76.2))
     (stroke (width 0) (type default) (color 0 0 0 0))
@@
     (stroke (width 0) (type default) (color 0 0 0 0))
   )
+  (wire (pts (xy 92.71 -17.78) (xy 92.71 -7.62))
+    (stroke (width 0) (type default) (color 0 0 0 0))
+  )
   (wire (pts (xy 429.26 83.82) (xy 429.26 104.14))
     (stroke (width 0) (type default) (color 0 0 0 0))
@@
     (stroke (width 0) (type default) (color 0 0 0 0))
   )
+  (wire (pts (xy 90.17 -7.62) (xy 85.09 -7.62))
+    (stroke (width 0) (type default) (color 0 0 0 0))
+  )
   (wire (pts (xy 129.54 236.22) (xy 133.35 236.22))
     (stroke (width 0) (type default) (color 0 0 0 0))
@@
     (stroke (width 0) (type default) (color 0 0 0 0))
   )
+  (wire (pts (xy 90.17 -7.62) (xy 92.71 -7.62))
+    (stroke (width 0) (type default) (color 0 0 0 0))
+  )
   (wire (pts (xy 80.01 120.65) (xy 80.01 121.92))
     (stroke (width 0) (type default) (color 0 0 0 0))
@@
     (stroke (width 0) (type default) (color 0 0 0 0))
   )
+  (wire (pts (xy 85.09 -10.16) (xy 85.09 -7.62))
+    (stroke (width 0) (type default) (color 0 0 0 0))
+  )
   (wire (pts (xy 393.7 26.67) (xy 402.59 26.67))
     (stroke (width 0) (type default) (color 0 0 0 0))
@@
     (stroke (width 0) (type default) (color 0 0 0 0))
   )
+  (wire (pts (xy 85.09 -81.28) (xy 91.44 -81.28))
+    (stroke (width 0) (type default) (color 0 0 0 0))
+  )
   (wire (pts (xy 31.75 64.77) (xy 30.48 64.77))
     (stroke (width 0) (type default) (color 0 0 0 0))
@@
     (stroke (width 0) (type default) (color 0 0 0 0))
   )
+  (wire (pts (xy 85.09 -22.86) (xy 90.17 -22.86))
+    (stroke (width 0) (type default) (color 0 0 0 0))
+  )
   (wire (pts (xy 15.24 67.31) (xy 15.24 74.93))
     (stroke (width 0) (type default) (color 0 0 0 0))
@@
     (stroke (width 0) (type default) (color 0 0 0 0))
   )
+  (wire (pts (xy 85.09 -66.04) (xy 92.71 -66.04))
+    (stroke (width 0) (type default) (color 0 0 0 0))
+  )
   (polyline (pts (xy 109.22 220.98) (xy 161.29 220.98))
     (stroke (width 0) (type default) (color 0 0 0 0))
@@
     (pin "2")
   )
+  (symbol (lib_id "Device:R") (at 90.17 -11.43 0) (unit 1)
+    (in_bom yes) (on_board yes) (fields_autoplaced)
+    (property "Reference" "R1" (id 0) (at 92.71 -12.7001 0)
+      (effects (font (size 1.27 1.27)) (justify left))
+    )
+    (property "Value" "1k" (id 1) (at 92.71 -10.1601 0)
+      (effects (font (size 1.27 1.27)) (justify left))
+    )
+    (property "Footprint" "" (id 2) (at 88.392 -11.43 90)
+      (effects (font (size 1.27 1.27)) hide)
+    )
+    (property "Datasheet" "~" (id 3) (at 90.17 -11.43 0)
+      (effects (font (size 1.27 1.27)) hide)
+    )
+    (pin "1")
+    (pin "2")
+  )
   (symbol (lib_id "Adafruit Ultimate GPS-eagle-import:LED0805") (at 229.87 69.85 180) (unit 1)
     (in_bom yes) (on_board yes)
@@
     (pin "2")
   )
+  (symbol (lib_id "Device:R") (at 90.17 -19.05 0) (unit 1)
+    (in_bom yes) (on_board yes) (fields_autoplaced)
+    (property "Reference" "R2" (id 0) (at 92.71 -20.3201 0)
+      (effects (font (size 1.27 1.27)) (justify left))
+    )
+    (property "Value" "4k" (id 1) (at 92.71 -17.7801 0)
+      (effects (font (size 1.27 1.27)) (justify left))
+    )
+    (property "Footprint" "" (id 2) (at 88.392 -19.05 90)
+      (effects (font (size 1.27 1.27)) hide)
+    )
+    (property "Datasheet" "~" (id 3) (at 90.17 -19.05 0)
+      (effects (font (size 1.27 1.27)) hide)
+    )
+    (pin "1")
+    (pin "2")
+  )
   (symbol (lib_id "power:+3V3") (at 92.71 -76.2 270) (unit 1)
     (in_bom yes) (on_board yes) (fields_autoplaced)
@@
     (pin "1")
   )
+  (symbol (lib_id "Device:R") (at 91.44 -77.47 0) (unit 1)
+    (in_bom yes) (on_board yes) (fields_autoplaced)
+    (property "Reference" "R2" (id 0) (at 93.98 -78.7401 0)
+      (effects (font (size 1.27 1.27)) (justify left))
+    )
+    (property "Value" "1.75k" (id 1) (at 93.98 -76.2001 0)
+      (effects (font (size 1.27 1.27)) (justify left))
+    )
+    (property "Footprint" "" (id 2) (at 89.662 -77.47 90)
+      (effects (font (size 1.27 1.27)) hide)
+    )
+    (property "Datasheet" "~" (id 3) (at 91.44 -77.47 0)
+      (effects (font (size 1.27 1.27)) hide)
+    )
+    (pin "1")
+    (pin "2")
+  )
   (symbol (lib_id "power:GND") (at 210.82 69.85 270) (unit 1)
     (in_bom yes) (on_board yes)
@@
     (pin "2")
   )
+  (symbol (lib_id "Device:R") (at 91.44 -69.85 0) (unit 1)
+    (in_bom yes) (on_board yes) (fields_autoplaced)
+    (property "Reference" "R1" (id 0) (at 93.98 -71.1201 0)
+      (effects (font (size 1.27 1.27)) (justify left))
+    )
+    (property "Value" "1k" (id 1) (at 93.98 -68.5801 0)
+      (effects (font (size 1.27 1.27)) (justify left))
+    )
+    (property "Footprint" "" (id 2) (at 89.662 -69.85 90)
+      (effects (font (size 1.27 1.27)) hide)
+    )
+    (property "Datasheet" "~" (id 3) (at 91.44 -69.85 0)
+      (effects (font (size 1.27 1.27)) hide)
+    )
+    (pin "1")
+    (pin "2")
+  )
   (symbol (lib_id "power:GND") (at 402.59 26.67 0) (unit 1)
     (in_bom yes) (on_board yes) (fields_autoplaced)
@@
       (reference "Q?") (unit 1) (value "FQP30N06L") (footprint "Package_TO_SOT_THT:TO-220-3_Vertical")
     )
+    (path "/329ddd32-68ca-44f0-84dd-4801bab1b487"
+      (reference "R1") (unit 1) (value "1k") (footprint "")
+    )
+    (path "/de9e7f12-1e66-412d-85a0-dee8a5a1031e"
+      (reference "R1") (unit 1) (value "1k") (footprint "")
+    )
+    (path "/4f66ab94-ccfa-4717-82b3-abea8a77ad56"
+      (reference "R2") (unit 1) (value "4k") (footprint "")
+    )
+    (path "/c9dd5558-90a0-4431-80e5-2c6dc5692e9a"
+      (reference "R2") (unit 1) (value "1.75k") (footprint "")
+    )
     (path "/1f95de38-c7d1-4c35-9a65-9314a6751ee0"

Commit message: ggg
Parts:
- removed C?: ???, symbol Device:C_Small
- removed C?: 330uF, symbol Device:C_Small
- removed C?: 100uF, symbol Device:C_Small
- removed D?: D_Schottky_Small, symbol Device:D_Schottky_Small
- removed L?: ???, symbol Device:L
- removed L?: 100uH, symbol Device:L
- removed R1 (x2): 1k, symbol Device:R
- removed R2: 4k, symbol Device:R
- removed R2: 1.75k, symbol Device:R
- removed U?: LM2576S-5, Package_TO_SOT_SMD:TO-263-5_TabPin3, symbol Regulator_Switching:LM2576S-5
- removed U?: LM2576S-3.3, Package_TO_SOT_SMD:TO-263-5_TabPin3, symbol Regulator_Switching:LM2576S-3.3
- added C?: 1000uF, symbol Device:C_Small
- added L?: 100uH, symbol Device:L
- added R? (x2): R, symbol Device:R
- added R?: 1Kohm, symbol Device:R
- added R?: 1.68Kohm, symbol Device:R
- added U?: LM2576S-ADJ, Package_TO_SOT_SMD:TO-263-5_TabPin3, symbol Regulator_Switching:LM2576S-ADJ
- C?: value ??? -> 1000uF
- L?: value ??? -> 100uH
Connections:
- net +3V3: now also C?.1, L?.2, R?.1; no longer C?.1, C?.1, C?.1, C?.1, C?.1, C?.1, C?.1, C?.1, C?.1, C?.1, C?.1, C?.1, C?.1, C?.1, C?.1, C?.1, C?.2, C?.2, C?.2, C?.2, C?.2, C?.2, C?.2, C?.2, C?.2, C?.2, C?.2, C?.2, C?.2, C?.2, C?.2, C?.2, C?.2, C?.2, C?.2, C?.2, C?.2, C?.2, C?.2, C?.2, C?.2, C?.2, D?.2 (A), D?.2 (A), J?.1 (Pin_1), J?.1 (Pin_1), J?.1 (Pin_1), J?.2 (Pin_2), J?.4 (Pin_4), J?.6 (VSS), J?.A1 (GND), J?.A12 (GND), J?.A4 (VBUS), J?.A9 (VBUS), J?.B1 (GND), J?.B12 (GND), J?.B4 (VBUS), J?.B9 (VBUS), L?.2, L?.2, Male?.1 (Pin_1), Male?.1 (Pin_1), Q?.3 (S), Q?.3 (S), R?.1, R?.1, R?.1, R?.1, R?.1, R?.2, R?.2, R?.2, R?.2, R?.2, R?.2, R?.2, SW?.1 (A), U?.1 (GND), U?.15 (GNDIO), U?.16 (GNDIO), U?.18 (COM2), U?.2 (GND), U?.23 (VSS), U?.25 (GNDIO), U?.3 (GND), U?.3 (VI), U?.32 (EXT_XOSC), U?.33 (GND_EP), U?.35 (VSS), U?.4 (FB), U?.47 (VSS), U?.49 (VSS), U?.5 (~{ON}/OFF), U?.7 (GND), U?.8 (VSSA), U?.P$12 (GND@3), U?.P$19 (GND@4), U?.P$3 (GND@1), U?.P$8 (GND@2), VDiv1_?.1, VDiv2_?.1, X?.2, X?.4, Y?.2, Y?.4
- net at C?.2, C?.2, J?.1 (Pin_1)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: now also U?.1 (VIN)
- net at D?.1 (K): now also L?.1, U?.2 (OUT)
- new net: R?.1, R?.2, U?.4 (FB) (x2)
- new net +6V: C?.1, J?.1 (Pin_1), J?.1 (Pin_1), J?.1 (Pin_1), L?.2, R?.1
- new net GND: C?.1, C?.1, C?.1, C?.1, C?.1, C?.1, C?.1, C?.1, C?.1, C?.1, C?.1, C?.1, C?.1, C?.1, C?.1, C?.2, C?.2, C?.2, C?.2, C?.2, C?.2, C?.2, C?.2, C?.2, C?.2, C?.2, C?.2, C?.2, C?.2, C?.2, C?.2, C?.2, C?.2, C?.2, C?.2, C?.2, C?.2, C?.2, C?.2, C?.2, C?.2, C?.2, D?.2 (A), D?.2 (A), J?.2 (Pin_2), J?.4 (Pin_4), J?.6 (VSS), J?.A1 (GND), J?.A12 (GND), J?.A4 (VBUS), J?.A9 (VBUS), J?.B1 (GND), J?.B12 (GND), J?.B4 (VBUS), J?.B9 (VBUS), L?.2, Male?.1 (Pin_1), Male?.1 (Pin_1), Q?.3 (S), Q?.3 (S), R?.1, R?.1, R?.1, R?.1, R?.1, R?.2, R?.2, R?.2, R?.2, R?.2, R?.2, R?.2, R?.2, R?.2, SW?.1 (A), U?.1 (GND), U?.15 (GNDIO), U?.16 (GNDIO), U?.18 (COM2), U?.2 (GND), U?.23 (VSS), U?.25 (GNDIO), U?.3 (GND), U?.3 (GND), U?.3 (VI), U?.32 (EXT_XOSC), U?.33 (GND_EP), U?.35 (VSS), U?.47 (VSS), U?.49 (VSS), U?.5 (~{ON}/OFF), U?.5 (~{ON}/OFF), U?.7 (GND), U?.8 (VSSA), U?.P$12 (GND@3), U?.P$19 (GND@4), U?.P$3 (GND@1), U?.P$8 (GND@2), VDiv1_?.1, VDiv2_?.1, X?.2, X?.4, Y?.2, Y?.4
Other:
- moved on the sheet: C?, D?, J?, L?, U?
